File: Trout-59.kicad_pcb (KiCad board)
At the start: 2 copper layers, 304.8 x 77.8 mm, 138 parts, among them SW1 SW_Push, U1 ATmega32U4-AU, U2 SRV05-4, Y1 16MHz

Commit message: Finalization
Crystal ground plane separated from main groung, gerber and BOM files finalized
Routing:
- net GND: track 191.4 -> 186.1 mm
Other:
- board text added: "Git - ProbablyNotAMoose |"
- board text added: "Layout inspired by UT47.2"
- board text removed: "Git - ProbablyNotAMoose | Layout inspired by UT47.2"
Changed lines of the file:
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@@
   (general
     (thickness 1.6)
-    (drawings 355)
-    (tracks 1038)
+    (drawings 356)
+    (tracks 1035)
     (zones 0)
     (modules 138)
@@
       (drillshape 0)
       (scaleselection 1)
-      (outputdirectory "Gerber/"))
+      (outputdirectory "BOM/"))
   )
   (net 0 "")
@@
     (tags capacitor)
     (attr smd)
-    (fp_text reference C2 (at -0.157154 -1.593995) (layer B.SilkS)
+    (fp_text reference C2 (at -0.157154 1.80975) (layer B.SilkS)
       (effects (font (size 1 1) (thickness 0.15)) (justify mirror))
     )
@@
     (tags "SMD SMT crystal")
     (attr smd)
-    (fp_text reference Y1 (at 0 2.45) (layer B.SilkS)
+    (fp_text reference Y1 (at 3.175 0) (layer B.SilkS)
       (effects (font (size 1 1) (thickness 0.15)) (justify mirror))
     )
@@
     )
   )
+  (gr_text "Layout inspired by UT47.2" (at 280.289 113.538) (layer B.SilkS)
+    (effects (font (size 1 1) (thickness 0.2)) (justify mirror))
+  )
   (gr_line (start 324.5 113.77496) (end 24.74965 113.77496) (layer Dwgs.User) (width 0.2))
   (gr_text Trout-59 (at 33.528 111.34725) (layer F.SilkS)
     (effects (font (size 2 2) (thickness 0.3)))
   )
-  (gr_text "Git - ProbablyNotAMoose | Layout inspired by UT47.2" (at 291.592 113.538) (layer B.SilkS)
+  (gr_text "Git - ProbablyNotAMoose | " (at 306.324 113.411) (layer B.SilkS)
     (effects (font (size 1.5 1.5) (thickness 0.25)) (justify mirror))
   )
@@
   (segment (start 95.912913 88.237087) (end 94.687691 88.237087) (width 0.381) (layer B.Cu) (net 2))
   (segment (start 89.417888 80.56312) (end 89.417888 80.753317) (width 0.381) (layer B.Cu) (net 2))
-  (segment (start 87.181663 72.362087) (end 88.138 73.318424) (width 0.381) (layer B.Cu) (net 2))
-  (segment (start 88.138 74.287326) (end 90.269087 76.418413) (width 0.381) (layer B.Cu) (net 2))
-  (segment (start 88.138 73.318424) (end 88.138 74.287326) (width 0.381) (layer B.Cu) (net 2))
   (segment (start 92.828077 86.377473) (end 90.39176 86.377473) (width 0.381) (layer B.Cu) (net 2))
   (segment (start 93.377686 86.927082) (end 92.828077 86.377473) (width 0.381) (layer B.Cu) (net 2))
@@
     (polygon
       (pts
-        (xy 98.425 85.725) (xy 86.51875 97.63125) (xy 74.6125 85.725) (xy 86.51875 73.81875)
-      )
-    )
-  )
-  (zone (net 2) (net_name GND) (layer B.Cu) (hatch edge 0.508)
-    (connect_pads (clearance 0.508))
-    (min_thickness 0.254)
-    (fill yes (arc_segments 32) (thermal_gap 0.508) (thermal_bridge_width 0.508))
-    (polygon
-      (pts
         (xy 88.9 45.24375) (xy 79.375 45.24375) (xy 79.375 38.1) (xy 88.9 38.1)
       )
     )
   )
-  (zone (net 2) (net_name GND) (layer B.Cu) (hatch edge 0.508)
+  (zone (net 2) (net_name GND) (layer F.Cu) (hatch edge 0.508)
     (connect_pads (clearance 0.508))
     (min_thickness 0.254)
@@
     (polygon
       (pts
-        (xy 96.8375 73.025) (xy 99.21875 73.025) (xy 99.21875 81.75625) (xy 94.45625 86.51875) (xy 83.34375 74.6125)
-        (xy 86.51875 71.4375) (xy 86.51875 66.675) (xy 90.4875 66.675)
+        (xy 327.025 115.8875) (xy 22.225 115.8875) (xy 22.225 38.1) (xy 327.025 38.1)
       )
     )
@@
       )
     )
-  )
-  (zone (net 2) (net_name GND) (layer F.Cu) (hatch edge 0.508)
-    (connect_pads (clearance 0.508))
-    (min_thickness 0.254)
-    (fill yes (arc_segments 32) (thermal_gap 0.508) (thermal_bridge_width 0.508))
     (polygon
       (pts
-        (xy 327.025 115.8875) (xy 22.225 115.8875) (xy 22.225 38.1) (xy 327.025 38.1)
+        (xy 90.297 71.12) (xy 89.535 71.882) (xy 89.535 79.502) (xy 91.821 81.788) (xy 95.631 81.788)
+        (xy 99.441 77.978) (xy 99.441 73.152) (xy 96.901 73.152) (xy 94.742 71.12)
       )
     )
   )
-  (zone (net 0) (net_name "") (layer B.Cu) (hatch edge 0.508)
+  (zone (net 2) (net_name GND) (layer B.Cu) (hatch edge 0.508)
     (connect_pads (clearance 0.508))
     (min_thickness 0.254)
-    (keepout (tracks allowed) (vias allowed) (copperpour not_allowed))
-    (fill (arc_segments 32) (thermal_gap 0.508) (thermal_bridge_width 0.508))
+    (fill yes (arc_segments 32) (thermal_gap 0.508) (thermal_bridge_width 0.508))
     (polygon
       (pts
-        (xy 96.774 73.025) (xy 99.187 73.025) (xy 99.187 81.788) (xy 98.806 81.788) (xy 98.806 73.279)
-        (xy 96.647 73.279) (xy 90.297 66.929) (xy 86.868 66.929) (xy 86.868 70.866) (xy 83.566 74.168)
-        (xy 94.615 85.725) (xy 98.679 81.788) (xy 98.933 82.042) (xy 94.615 86.36) (xy 83.058 74.168)
-        (xy 86.487 70.739) (xy 86.487 66.675) (xy 90.424 66.675)
+        (xy 96.52 73.279) (xy 99.06 73.279) (xy 99.06 77.724) (xy 95.377 81.407) (xy 91.948 81.407)
+        (xy 89.789 79.248) (xy 89.789 71.882) (xy 90.297 71.374) (xy 94.615 71.374)
       )
     )
