File: Trout-59.sch (KiCad schematic (older format))
At the start: 137 parts, among them SW1 SW_Push, U1 ATmega32U4-AU, U2 SRV05-4, Y1 16MHz

Commit message: Finalization
Crystal ground plane separated from main groung, gerber and BOM files finalized
Parts:
- U2: C-Code (none) -> C85364
Changed lines of the file:
@@
 F 2 "Package_TO_SOT_SMD:SOT-23-6" H 11400 7400 50  0001 C CNN
 F 3 "http://www.onsemi.com/pub/Collateral/SRV05-4-D.PDF" H 10700 7850 50  0001 C CNN
-F 4 "" H 10700 7850 50  0001 C CNN "C-Code"
+F 4 "C85364" H 10700 7850 50  0001 C CNN "C-Code"
 	1    10700 7850
 	1    0    0    -1
